File: hard_cam_usb/hard_cam_usb.kicad_pcb (KiCad board)
At the start: 2 copper layers, 33.3 x 80.6 mm, 2 parts, among them J1 FFC-FPC Conn, J2 USB_B_Mini

Commit message: sent to production
Parts:
- added H1: MountingHole_Pad, MountingHole:MountingHole_3.2mm_M3_Pad_Via, F.Cu at (65.2, 147.8)
- added H2: MountingHole_Pad, MountingHole:MountingHole_3.2mm_M3_Pad_Via, F.Cu at (65.2, 171.7)
- added H3: MountingHole_Pad, MountingHole:MountingHole_3.2mm_M3_Pad_Via, F.Cu at (184.6, 147.8)
- added H4: MountingHole_Pad, MountingHole:MountingHole_3.2mm_M3_Pad_Via, F.Cu at (184.6, 171.7)
- added H5: MountingHole_Pad, MountingHole:MountingHole_3.2mm_M3_Pad_Via, F.Cu at (313.0, 217.1)
- added H6: MountingHole_Pad, MountingHole:MountingHole_3.2mm_M3_Pad_Via, F.Cu at (357.7, 206.7)
- added H7: MountingHole_Pad, MountingHole:MountingHole_3.2mm_M3_Pad_Via, F.Cu at (172.6, 210.6)
- added H8: MountingHole_Pad, MountingHole:MountingHole_3.2mm_M3_Pad_Via, F.Cu at (337.5, 235.0)
- added J3: FFC-FPC Conn, 59453-051110ECHLF:59453051110ECHLF, F.Cu at (288.7, 209.7)
- added J4: Mini B USB - Vertical, Hard_PLM:MUSB-B5-S-VT-TSMT-TR, F.Cu at (352.8, 237.0)
- added J5: FFC-FPC Conn, 59453-051110ECHLF:59453051110ECHLF, F.Cu at (171.8, 155.0)
- added J6: Mini B USB - Vertical, Hard_PLM:MUSB-B5-S-VT-TSMT-TR, F.Cu at (169.4, 224.9)
- added L1: Logo-logo, LED_driver_PCB:logo_vulcur, F.Cu at (61.5, 159.8)
- added L2: Logo-logo, LED_driver_PCB:logo_vulcur, F.Cu at (180.0, 160.7)
- added L3: Logo-logo, LED_driver_PCB:logo_vulcur, F.Cu at (348.0, 215.4)
- moved J2 140.5 mm to (48.5, 171.5)
- moved J1 137.2 mm to (52.4, 155.0)
Routing:
- net VCC: track 0.00 -> 167.0 mm, vias 0 -> 12
- net /id2: track 0.00 -> 80.5 mm, vias 0 -> 8
- net /D2_-: track 0.00 -> 79.0 mm, vias 0 -> 2
- net /D2_+: track 0.00 -> 78.8 mm, vias 0 -> 2
- net /id3: track 0.00 -> 72.8 mm, vias 0 -> 2
- net /D3_-: track 0.00 -> 72.1 mm, vias 0 -> 2
- net /D3_+: track 0.00 -> 72.1 mm, vias 0 -> 2
- net GND: track 0.00 -> 23.9 mm, vias 0 -> 191
- net /id: track 0.00 -> 14.9 mm, vias 0 -> 2
- net /D+: track 0.00 -> 14.7 mm, vias 0 -> 2
- net /D-: track 0.00 -> 14.7 mm, vias 0 -> 2
- added copper zone on B.Cu, net GND
- added copper zone on F.Cu, net GND
- added copper zone on In1.Cu, net GND
- added copper zone on In2.Cu, net GND
- added copper zone on B.Cu, net VCC
Other:
- board size 33.3 x 80.6 mm -> 322.3 x 96.8 mm
- copper layers 2 -> 4
- net class 24V added: clearance 0.3048, trace_width 0.381, via_dia 0.635, via_drill 0.3302
- net class Default: via_dia 0.8 -> 0.508; via_drill 0.4 -> 0.254
- rule pad_to_mask_clearance: 0 -> 0.2
- rule trace_min: 0.2 -> 0.1778
- rule via_min_drill: 0.3 -> 0.254
- rule via_min_size: 0.4 -> 0.508
- board text added: "Must be manufacturer with JLC7628 PCB stackup"
- board text added: "cam_usb_1.1"
- board text added: "cam_usb_1.2"
- board text added: "cam_usb_1.3"
